File: ESP32.kicad_pcb (KiCad board)
At the start: 4 copper layers, 42.7 x 59.8 mm, 53 parts, among them J1 USB_B_Micro, J2 Conn_01x18_Male, J3 Conn_01x18_Male, Q1 AO3401A, Q2 BC847, Q3 BC847, SW1 SW_MEC_5E, U1 ESP32-WROOM-32, U2 MCP73831-2-OT, U3 CP2104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

Commit message: x
Routing:
- net /D+: track 32.5 -> 31.9 mm
